File: c-pro-micro.kicad_pcb (KiCad board)
At the start: 2 copper layers, 17.8 x 33 mm, 23 parts, among them J1 USB_C_Receptacle, J2 Conn_01x12, J3 Conn_01x12, U1 ATmega32U4, Y1 16MHz

Commit message: Rev2
Parts:
- added D4: RB161MM-20, Diode_SMD:D_SOD-123F, F.Cu at (110.9, 129.8)
- C1: footprint Capacitors_SMD:C_0603 -> Capacitor_SMD:C_0603_1608Metric
- C2: footprint Capacitors_SMD:C_0603 -> Capacitor_SMD:C_0402_1005Metric
- C3, C4, C5, C6: footprint Capacitors_SMD:C_0402 -> Capacitor_SMD:C_0402_1005Metric
- D1, D2, D3: footprint LEDs:LED_0603 -> LED_SMD:LED_0603_1608Metric
- F1: footprint Fuse_Holders_and_Fuses:Fuse_SMD1206_Reflow -> Fuse:Fuse_1206_3216Metric
- J1: footprint Connectors_USB:USB_C_Receptacle_Amphenol_12401610E4-2A -> Connector_USB:USB_C_Receptacle_Amphenol_12401610E4-2A
- J2: footprint Pin_Headers:Pin_Header_Straight_1x12 -> guri-lib:ProMicro_LeftPinhead
- J3: footprint Pin_Headers:Pin_Header_Straight_1x12 -> guri-lib:ProMicro_RightPinhead
- R1, R2: footprint Resistors_SMD:R_0603 -> Resistor_SMD:R_0402_1005Metric; moved to F.Cu
- R3, R4, R5, R6: footprint Resistors_SMD:R_0402 -> Resistor_SMD:R_0402_1005Metric
- R7, R8: footprint Resistors_SMD:R_0603 -> Resistor_SMD:R_0402_1005Metric
- Y1: footprint Crystals:Crystal_SMD_SeikoEpson_FA238-4pin_3.2x2.5mm -> Crystal:Crystal_SMD_SeikoEpson_FA238-4Pin_3.2x2.5mm
- moved R1 6.38 mm to (109.1, 128.6), turned to 90 degrees
- moved R2 6.22 mm to (106.3, 128.4), turned to 90 degrees
- moved R4 4.74 mm to (105.8, 132.2)
- moved R3 3.27 mm to (107.2, 132.0)
- moved C1 2.75 mm to (108.7, 131.0)
- moved D1 2.57 mm to (104.0, 131.1), turned to 90 degrees
- moved R5 1.50 mm to (104.0, 128.5), turned to 270 degrees
- moved R7 0.87 mm to (105.2, 148.4), turned to 270 degrees
- moved R8 0.87 mm to (112.8, 148.4), turned to 270 degrees
- moved C2 0.78 mm to (104.5, 134.0), turned to 180 degrees
- moved F1 0.25 mm to (113.5, 129.8)
Connections:
- F1 pad 1: VCC -> Net-(D4-Pad2)
- U1 pad 7: VCC -> VBUS
Routing:
- net VBUS: track 13.9 -> 28.6 mm, vias 0 -> 2
- net VCC: track 68.9 -> 81.5 mm, vias 6 -> 5
- net RESET: track 26.9 -> 37.7 mm
- net GND: track 75.3 -> 66.1 mm, vias 21 -> 18
- net Net-(J1-PadA6): track 4.15 -> 9.18 mm
- net Net-(J1-PadA5): track 7.42 -> 2.42 mm, vias 1 -> 0
- net Net-(J1-PadB5): track 1.83 -> 6.65 mm, vias 1 -> 2
- net Net-(J1-PadA7): track 7.93 -> 12.4 mm, vias 2 -> 3
- net D+: track 7.22 -> 3.20 mm
- net D-: track 6.49 -> 2.59 mm, vias 2 -> 0
- net Net-(D4-Pad2): track 0.00 -> 2.61 mm
- net Net-(D3-Pad1): track 2.90 -> 1.78 mm
- net Net-(C2-Pad1): track 2.02 -> 2.91 mm
- net Net-(R7-Pad2): track 14.7 -> 15.6 mm
- net D4: track 16.5 -> 15.6 mm
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Other:
- board text added: "@zgtk-guri"
- board text added: "C-Pro Micro R2"
