File: c-pro-micro.kicad_pcb (KiCad board)
At the start: 2 copper layers, 17.8 x 33 mm, 24 parts, among them J1 USB_C_Receptacle, J2 Conn_01x12, J3 Conn_01x12, U1 ATmega32U4, Y1 16MHz

Commit message: Rev3
Parts:
- J1: footprint Connector_USB:USB_C_Receptacle_Amphenol_12401610E4-2A -> guri-lib:CX90M-16P
- moved J1 2.00 mm to (108.9, 119.0)
Connections:
- J1 pad A8: Net-(J1-PadA8) -> (no net)
- J1 pad B8: Net-(J1-PadB8) -> (no net)
- U1 pad 12: Net-(U1-Pad12) -> (no net)
- U1 pad 26: Net-(U1-Pad26) -> (no net)
- U1 pad 32: Net-(U1-Pad32) -> (no net)
- U1 pad 40: Net-(U1-Pad40) -> (no net)
- U1 pad 41: Net-(U1-Pad41) -> (no net)
Routing:
- net GND: track 66.1 -> 44.9 mm, vias 18 -> 20
- net VBUS: track 28.6 -> 35.9 mm, vias 2 -> 3
- net Net-(J1-PadA6): track 9.18 -> 16.0 mm, vias 0 -> 2
- net VCC: track 81.5 -> 75.7 mm
- net RESET: track 37.7 -> 32.2 mm
- net Net-(J1-PadA5): track 2.42 -> 5.95 mm
- net Net-(J1-PadA7): track 12.4 -> 14.3 mm, vias 3 -> 2
- net Net-(J1-PadB5): track 6.65 -> 5.82 mm, vias 2 -> 0
Other:
- outline, holes or cut-outs redrawn
- board text added: "C-Pro Micro R3"
- board text removed: "C-Pro Micro R2"
