File: c-pro-micro.sch (KiCad schematic (older format))
At the start: 23 parts, among them J1 USB_C_Receptacle, J2 Conn_01x12, J3 Conn_01x12, U1 ATmega32U4, Y1 16MHz

Commit message: add parts informations
Parts:
- C1: footprint (none) -> Capacitors_SMD:C_0805; ElecrowPN (none) -> 2015010A
- C2: footprint (none) -> Capacitors_SMD:C_0603; ElecrowPN (none) -> 2013501A
- C3, C4: footprint (none) -> Capacitors_SMD:C_0603; ElecrowPN (none) -> 2010822A
- C5, C6: footprint (none) -> Capacitors_SMD:C_0603; ElecrowPN (none) -> 2013010A
- D1: footprint (none) -> LEDs:LED_0603; ElecrowPN (none) -> 4040506A
- D2: footprint (none) -> LEDs:LED_0603; ElecrowPN (none) -> 4040606A
- D3: footprint (none) -> LEDs:LED_0603; ElecrowPN (none) -> 4040706A
- F1: value Polyfuse -> 500mA; footprint (none) -> Fuse_Holders_and_Fuses:Fuse_SMD1206_Reflow; ElecrowPN (none) -> 4060505A
- J1: footprint (none) -> Connectors_USB:USB_C_Receptacle_Amphenol_12401610E4-2A; DigikeyPN (none) -> WM12856CT-ND; MF (none) -> Molex; MPN (none) -> 1054500101
- J2, J3: footprint (none) -> Pin_Headers:Pin_Header_Straight_1x12
- R1, R2: footprint (none) -> Resistors_SMD:R_0603; MPN (none) -> 0603WAF5101T5E
- R3, R4: footprint (none) -> Resistors_SMD:R_0603; MPN (none) -> 0603WAF220JT5E
- R5: footprint (none) -> Resistors_SMD:R_0603; ElecrowPN (none) -> 1022501A
- R6: footprint (none) -> Resistors_SMD:R_0603; ElecrowPN (none) -> 1023510A
- R7, R8: footprint (none) -> Resistors_SMD:R_0603; ElecrowPN (none) -> 1021633A
- U1: footprint (none) -> Housings_DFN_QFN:QFN-44-1EP_7x7mm_Pitch0.5mm; DigikeyPN (none) -> ATMEGA32U4-MURCT-ND; MF (none) -> Atmel; MPN (none) -> ATMEGA32U4-MUR
- Y1: footprint (none) -> Crystals:Crystal_SMD_SeikoEpson_FA238-4pin_3.2x2.5mm; DigikeyPN (none) -> SER3686CT-ND; MF (none) -> EPSON; MPN (none) -> FA-238 16.0000MB-C3
Changed lines of the file:
@@
 LIBS:contrib
 LIBS:valves
+LIBS:c-pro-micro-cache
 EELAYER 25 0
 EELAYER END
@@
 F 0 "U1" H 6000 5000 50  0000 C CNN
 F 1 "ATmega32U4" H 6250 1750 50  0000 C CNN
-F 2 "" H 8100 4400 50  0001 C CNN
+F 2 "Housings_DFN_QFN:QFN-44-1EP_7x7mm_Pitch0.5mm" H 8100 4400 50  0001 C CNN
 F 3 "" H 8100 4400 50  0001 C CNN
+F 4 "Atmel" H 6900 3300 60  0001 C CNN "MF"
+F 5 "ATMEGA32U4-MUR" H 6900 3300 60  0001 C CNN "MPN"
+F 6 "ATMEGA32U4-MURCT-ND" H 6900 3300 60  0001 C CNN "DigikeyPN"
 	1    6900 3300
 	1    0    0    -1
@@
 F 0 "J1" H 1150 4950 50  0000 L CNN
 F 1 "USB_C_Receptacle" H 1950 4950 50  0000 R CNN
-F 2 "" H 1700 3500 50  0001 C CNN
+F 2 "Connectors_USB:USB_C_Receptacle_Amphenol_12401610E4-2A" H 1700 3500 50  0001 C CNN
 F 3 "" H 1700 3500 50  0001 C CNN
+F 4 "Molex" H 1550 3500 60  0001 C CNN "MF"
+F 5 "1054500101" H 1550 3500 60  0001 C CNN "MPN"
+F 6 "WM12856CT-ND" H 1550 3500 60  0001 C CNN "DigikeyPN"
 	1    1550 3500
 	1    0    0    -1
@@
 F 0 "R2" V 2580 2800 50  0000 C CNN
 F 1 "5.1k" V 2500 2800 50  0000 C CNN
-F 2 "" V 2430 2800 50  0001 C CNN
+F 2 "Resistors_SMD:R_0603" V 2430 2800 50  0001 C CNN
 F 3 "" H 2500 2800 50  0001 C CNN
+F 4 "0603WAF5101T5E" V 2500 2800 60  0001 C CNN "MPN"
 	1    2500 2800
 	0    1    1    0
@@
 F 0 "R1" V 2580 2700 50  0000 C CNN
 F 1 "5.1k" V 2500 2700 50  0000 C CNN
-F 2 "" V 2430 2700 50  0001 C CNN
+F 2 "Resistors_SMD:R_0603" V 2430 2700 50  0001 C CNN
 F 3 "" H 2500 2700 50  0001 C CNN
+F 4 "0603WAF5101T5E" V 2500 2700 60  0001 C CNN "MPN"
 	1    2500 2700
 	0    1    -1   0
@@
 F 0 "R4" V 2580 3200 50  0000 C CNN
 F 1 "22" V 2500 3200 50  0000 C CNN
-F 2 "" V 2430 3200 50  0001 C CNN
+F 2 "Resistors_SMD:R_0603" V 2430 3200 50  0001 C CNN
 F 3 "" H 2500 3200 50  0001 C CNN
+F 4 "0603WAF220JT5E" V 2500 3200 60  0001 C CNN "MPN"
 	1    2500 3200
 	0    1    1    0
@@
 F 0 "R3" V 2580 3100 50  0000 C CNN
 F 1 "22" V 2500 3100 50  0000 C CNN
-F 2 "" V 2430 3100 50  0001 C CNN
+F 2 "Resistors_SMD:R_0603" V 2430 3100 50  0001 C CNN
 F 3 "" H 2500 3100 50  0001 C CNN
+F 4 "0603WAF220JT5E" V 2500 3100 60  0001 C CNN "MPN"
 	1    2500 3100
 	0    1    -1   0
@@
 F 0 "C5" H 5025 2450 50  0000 L CNN
 F 1 "0.1u" H 5025 2250 50  0000 L CNN
-F 2 "" H 5038 2200 50  0001 C CNN
+F 2 "Capacitors_SMD:C_0603" H 5038 2200 50  0001 C CNN
 F 3 "" H 5000 2350 50  0001 C CNN
+F 4 "2013010A" H 5000 2350 60  0001 C CNN "ElecrowPN"
 	1    5000 2350
 	1    0    0    -1
@@
 F 0 "C2" H 4625 3050 50  0000 L CNN
 F 1 "1u" H 4625 2850 50  0000 L CNN
-F 2 "" H 4638 2800 50  0001 C CNN
+F 2 "Capacitors_SMD:C_0603" H 4638 2800 50  0001 C CNN
 F 3 "" H 4600 2950 50  0001 C CNN
+F 4 "2013501A" H 4600 2950 60  0001 C CNN "ElecrowPN"
 	1    4600 2950
 	1    0    0    -1
@@
 F 0 "R6" V 5180 3150 50  0000 C CNN
 F 1 "10k" V 5100 3150 50  0000 C CNN
-F 2 "" V 5030 3150 50  0001 C CNN
+F 2 "Resistors_SMD:R_0603" V 5030 3150 50  0001 C CNN
 F 3 "" H 5100 3150 50  0001 C CNN
+F 4 "1023510A" V 5100 3150 60  0001 C CNN "ElecrowPN"
 	1    5100 3150
 	0    -1   -1   0
@@
 P 2900 2300
 F 0 "F1" V 2800 2300 50  0000 C CNN
-F 1 "Polyfuse" V 3000 2300 50  0000 C CNN
-F 2 "" H 2950 2100 50  0001 L CNN
+F 1 "500mA" V 3000 2300 50  0000 C CNN
+F 2 "Fuse_Holders_and_Fuses:Fuse_SMD1206_Reflow" H 2950 2100 50  0001 L CNN
 F 3 "" H 2900 2300 50  0001 C CNN
+F 4 "4060505A" V 2900 2300 60  0001 C CNN "ElecrowPN"
 	1    2900 2300
 	0    1    1    0
@@
 F 0 "Y1" V 5300 3700 50  0000 L CNN
 F 1 "16MHz" V 5400 3700 50  0000 L CNN
-F 2 "" H 5050 3800 50  0001 C CNN
+F 2 "Crystals:Crystal_SMD_SeikoEpson_FA238-4pin_3.2x2.5mm" H 5050 3800 50  0001 C CNN
 F 3 "" H 5050 3800 50  0001 C CNN
+F 4 "EPSON" V 5050 3800 60  0001 C CNN "MF"
+F 5 "FA-238 16.0000MB-C3" V 5050 3800 60  0001 C CNN "MPN"
+F 6 "SER3686CT-ND" V 5050 3800 60  0001 C CNN "DigikeyPN"
 	1    5050 3800
 	0    1    1    0
@@
 F 0 "C3" H 4725 3700 50  0000 L CNN
 F 1 "22p" H 4725 3500 50  0000 L CNN
-F 2 "" H 4738 3450 50  0001 C CNN
+F 2 "Capacitors_SMD:C_0603" H 4738 3450 50  0001 C CNN
 F 3 "" H 4700 3600 50  0001 C CNN
+F 4 "2010822A" H 4700 3600 60  0001 C CNN "ElecrowPN"
 	1    4700 3600
 	0    1    1    0
@@
 F 0 "C4" H 4725 4100 50  0000 L CNN
 F 1 "22p" H 4725 3900 50  0000 L CNN
-F 2 "" H 4738 3850 50  0001 C CNN
+F 2 "Capacitors_SMD:C_0603" H 4738 3850 50  0001 C CNN
 F 3 "" H 4700 4000 50  0001 C CNN
+F 4 "2010822A" H 4700 4000 60  0001 C CNN "ElecrowPN"
 	1    4700 4000
 	0    1    1    0
@@
 F 0 "R8" V 8830 3200 50  0000 C CNN
 F 1 "330" V 8750 3200 50  0000 C CNN
-F 2 "" V 8680 3200 50  0001 C CNN
+F 2 "Resistors_SMD:R_0603" V 8680 3200 50  0001 C CNN
 F 3 "" H 8750 3200 50  0001 C CNN
+F 4 "1021633A" V 8750 3200 60  0001 C CNN "ElecrowPN"
 	1    8750 3200
 	1    0    0    -1
@@
 F 0 "D3" H 8750 2900 50  0000 C CNN
 F 1 "Green" H 8750 2700 50  0000 C CNN
-F 2 "" H 8750 2800 50  0001 C CNN
+F 2 "LEDs:LED_0603" H 8750 2800 50  0001 C CNN
 F 3 "" H 8750 2800 50  0001 C CNN
+F 4 "4040706A" H 8750 2800 60  0001 C CNN "ElecrowPN"
 	1    8750 2800
 	0    -1   -1   0
@@
 F 0 "D1" H 3300 4150 50  0000 C CNN
 F 1 "Red" H 3300 3950 50  0000 C CNN
-F 2 "" H 3300 4050 50  0001 C CNN
+F 2 "LEDs:LED_0603" H 3300 4050 50  0001 C CNN
 F 3 "" H 3300 4050 50  0001 C CNN
+F 4 "4040506A" H 3300 4050 60  0001 C CNN "ElecrowPN"
 	1    3300 4050
 	0    -1   -1   0
@@
 F 0 "R5" V 3380 3650 50  0000 C CNN
 F 1 "1k" V 3300 3650 50  0000 C CNN
-F 2 "" V 3230 3650 50  0001 C CNN
+F 2 "Resistors_SMD:R_0603" V 3230 3650 50  0001 C CNN
 F 3 "" H 3300 3650 50  0001 C CNN
+F 4 "1022501A" V 3300 3650 60  0001 C CNN "ElecrowPN"
 	1    3300 3650
 	1    0    0    -1
@@
 F 0 "C1" H 3175 2650 50  0000 L CNN
 F 1 "10u" H 3175 2450 50  0000 L CNN
-F 2 "" H 3188 2400 50  0001 C CNN
+F 2 "Capacitors_SMD:C_0805" H 3188 2400 50  0001 C CNN
 F 3 "" H 3150 2550 50  0001 C CNN
+F 4 "2015010A" H 3150 2550 60  0001 C CNN "ElecrowPN"
 	1    3150 2550
 	1    0    0    -1
@@
 F 0 "C6" H 5125 1800 50  0000 L CNN
 F 1 "0.1u" H 5125 1600 50  0000 L CNN
-F 2 "" H 5138 1550 50  0001 C CNN
+F 2 "Capacitors_SMD:C_0603" H 5138 1550 50  0001 C CNN
 F 3 "" H 5100 1700 50  0001 C CNN
+F 4 "2013010A" H 5100 1700 60  0001 C CNN "ElecrowPN"
 	1    5100 1700
 	1    0    0    -1
@@
 F 0 "J3" H 4100 6550 50  0000 C CNN
 F 1 "Conn_01x12" H 4100 5250 50  0000 C CNN
-F 2 "" H 4100 5950 50  0001 C CNN
+F 2 "Pin_Headers:Pin_Header_Straight_1x12" H 4100 5950 50  0001 C CNN
 F 3 "" H 4100 5950 50  0001 C CNN
 	1    4100 5950
@@
 F 0 "J2" H 2600 6650 50  0000 C CNN
 F 1 "Conn_01x12" H 2600 5350 50  0000 C CNN
-F 2 "" H 2600 6050 50  0001 C CNN
+F 2 "Pin_Headers:Pin_Header_Straight_1x12" H 2600 6050 50  0001 C CNN
 F 3 "" H 2600 6050 50  0001 C CNN
 	1    2600 6050
@@
 F 0 "R7" V 8530 1500 50  0000 C CNN
 F 1 "330" V 8450 1500 50  0000 C CNN
-F 2 "" V 8380 1500 50  0001 C CNN
+F 2 "Resistors_SMD:R_0603" V 8380 1500 50  0001 C CNN
 F 3 "" H 8450 1500 50  0001 C CNN
+F 4 "1021633A" V 8450 1500 60  0001 C CNN "ElecrowPN"
 	1    8450 1500
 	1    0    0    -1
@@
 F 0 "D2" H 8450 1200 50  0000 C CNN
 F 1 "Yellow" H 8450 1000 50  0000 C CNN
-F 2 "" H 8450 1100 50  0001 C CNN
+F 2 "LEDs:LED_0603" H 8450 1100 50  0001 C CNN
 F 3 "" H 8450 1100 50  0001 C CNN
+F 4 "4040606A" H 8450 1100 60  0001 C CNN "ElecrowPN"
 	1    8450 1100
 	0    -1   -1   0

Commit message: Change components footprint
Parts:
- C1: footprint Capacitors_SMD:C_0805 -> Capacitors_SMD:C_0603; ElecrowPN 2015010A -> (none); MPN (none) -> CL10A106KP8NNNC
- C3, C4: footprint Capacitors_SMD:C_0603 -> Capacitors_SMD:C_0402; ElecrowPN 2010822A -> (none); MPN (none) -> 0402CG220J500NT
- C5, C6: footprint Capacitors_SMD:C_0603 -> Capacitors_SMD:C_0402; ElecrowPN 2013010A -> (none); MPN (none) -> CL05B104KO5NNNC
- J1: DigikeyPN WM12856CT-ND -> 12401610E4#2ACT-ND; MF Molex -> Amphenol Commercial Products; MPN 1054500101 -> 12401610E4#2A
- R3, R4: footprint Resistors_SMD:R_0603 -> Resistors_SMD:R_0402; MPN 0603WAF220JT5E -> 0402WGF220JTCE
- R5: footprint Resistors_SMD:R_0603 -> Resistors_SMD:R_0402; ElecrowPN 1022501A -> (none); MPN (none) -> 0402WGF1001TCE
- R6: footprint Resistors_SMD:R_0603 -> Resistors_SMD:R_0402; ElecrowPN 1023510A -> (none); MPN (none) -> 0402WGF1002TCE
- U1: footprint Housings_DFN_QFN:QFN-44-1EP_7x7mm_Pitch0.5mm -> guri-lib:QFN-44-1EP_7x7mm_Pitch0.5mm_without_bottom
Changed lines of the file:
@@
 F 0 "U1" H 6000 5000 50  0000 C CNN
 F 1 "ATmega32U4" H 6250 1750 50  0000 C CNN
-F 2 "Housings_DFN_QFN:QFN-44-1EP_7x7mm_Pitch0.5mm" H 8100 4400 50  0001 C CNN
+F 2 "guri-lib:QFN-44-1EP_7x7mm_Pitch0.5mm_without_bottom" H 8100 4400 50  0001 C CNN
 F 3 "" H 8100 4400 50  0001 C CNN
 F 4 "Atmel" H 6900 3300 60  0001 C CNN "MF"
@@
 F 2 "Connectors_USB:USB_C_Receptacle_Amphenol_12401610E4-2A" H 1700 3500 50  0001 C CNN
 F 3 "" H 1700 3500 50  0001 C CNN
-F 4 "Molex" H 1550 3500 60  0001 C CNN "MF"
-F 5 "1054500101" H 1550 3500 60  0001 C CNN "MPN"
-F 6 "WM12856CT-ND" H 1550 3500 60  0001 C CNN "DigikeyPN"
+F 4 "Amphenol Commercial Products" H 1550 3500 60  0001 C CNN "MF"
+F 5 "12401610E4#2A" H 1550 3500 60  0001 C CNN "MPN"
+F 6 "12401610E4#2ACT-ND" H 1550 3500 60  0001 C CNN "DigikeyPN"
 	1    1550 3500
 	1    0    0    -1
@@
 F 0 "R4" V 2580 3200 50  0000 C CNN
 F 1 "22" V 2500 3200 50  0000 C CNN
-F 2 "Resistors_SMD:R_0603" V 2430 3200 50  0001 C CNN
+F 2 "Resistors_SMD:R_0402" V 2430 3200 50  0001 C CNN
 F 3 "" H 2500 3200 50  0001 C CNN
-F 4 "0603WAF220JT5E" V 2500 3200 60  0001 C CNN "MPN"
+F 4 "0402WGF220JTCE" V 2500 3200 60  0001 C CNN "MPN"
 	1    2500 3200
 	0    1    1    0
@@
 F 0 "R3" V 2580 3100 50  0000 C CNN
 F 1 "22" V 2500 3100 50  0000 C CNN
-F 2 "Resistors_SMD:R_0603" V 2430 3100 50  0001 C CNN
+F 2 "Resistors_SMD:R_0402" V 2430 3100 50  0001 C CNN
 F 3 "" H 2500 3100 50  0001 C CNN
-F 4 "0603WAF220JT5E" V 2500 3100 60  0001 C CNN "MPN"
+F 4 "0402WGF220JTCE" V 2500 3100 60  0001 C CNN "MPN"
 	1    2500 3100
 	0    1    -1   0
@@
 F 0 "C5" H 5025 2450 50  0000 L CNN
 F 1 "0.1u" H 5025 2250 50  0000 L CNN
-F 2 "Capacitors_SMD:C_0603" H 5038 2200 50  0001 C CNN
+F 2 "Capacitors_SMD:C_0402" H 5038 2200 50  0001 C CNN
 F 3 "" H 5000 2350 50  0001 C CNN
-F 4 "2013010A" H 5000 2350 60  0001 C CNN "ElecrowPN"
+F 4 "CL05B104KO5NNNC" H 5000 2350 60  0001 C CNN "MPN"
 	1    5000 2350
 	1    0    0    -1
@@
 F 0 "R6" V 5180 3150 50  0000 C CNN
 F 1 "10k" V 5100 3150 50  0000 C CNN
-F 2 "Resistors_SMD:R_0603" V 5030 3150 50  0001 C CNN
+F 2 "Resistors_SMD:R_0402" V 5030 3150 50  0001 C CNN
 F 3 "" H 5100 3150 50  0001 C CNN
-F 4 "1023510A" V 5100 3150 60  0001 C CNN "ElecrowPN"
+F 4 "0402WGF1002TCE" V 5100 3150 60  0001 C CNN "MPN"
 	1    5100 3150
 	0    -1   -1   0
@@
 F 0 "C3" H 4725 3700 50  0000 L CNN
 F 1 "22p" H 4725 3500 50  0000 L CNN
-F 2 "Capacitors_SMD:C_0603" H 4738 3450 50  0001 C CNN
+F 2 "Capacitors_SMD:C_0402" H 4738 3450 50  0001 C CNN
 F 3 "" H 4700 3600 50  0001 C CNN
-F 4 "2010822A" H 4700 3600 60  0001 C CNN "ElecrowPN"
+F 4 "0402CG220J500NT" H 4700 3600 60  0001 C CNN "MPN"
 	1    4700 3600
 	0    1    1    0
@@
 F 0 "C4" H 4725 4100 50  0000 L CNN
 F 1 "22p" H 4725 3900 50  0000 L CNN
-F 2 "Capacitors_SMD:C_0603" H 4738 3850 50  0001 C CNN
+F 2 "Capacitors_SMD:C_0402" H 4738 3850 50  0001 C CNN
 F 3 "" H 4700 4000 50  0001 C CNN
-F 4 "2010822A" H 4700 4000 60  0001 C CNN "ElecrowPN"
+F 4 "0402CG220J500NT" H 4700 4000 60  0001 C CNN "MPN"
 	1    4700 4000
 	0    1    1    0
@@
 F 0 "R5" V 3380 3650 50  0000 C CNN
 F 1 "1k" V 3300 3650 50  0000 C CNN
-F 2 "Resistors_SMD:R_0603" V 3230 3650 50  0001 C CNN
+F 2 "Resistors_SMD:R_0402" V 3230 3650 50  0001 C CNN
 F 3 "" H 3300 3650 50  0001 C CNN
-F 4 "1022501A" V 3300 3650 60  0001 C CNN "ElecrowPN"
+F 4 "0402WGF1001TCE" V 3300 3650 60  0001 C CNN "MPN"
 	1    3300 3650
 	1    0    0    -1
@@
 F 0 "C1" H 3175 2650 50  0000 L CNN
 F 1 "10u" H 3175 2450 50  0000 L CNN
-F 2 "Capacitors_SMD:C_0805" H 3188 2400 50  0001 C CNN
+F 2 "Capacitors_SMD:C_0603" H 3188 2400 50  0001 C CNN
 F 3 "" H 3150 2550 50  0001 C CNN
-F 4 "2015010A" H 3150 2550 60  0001 C CNN "ElecrowPN"
+F 4 "CL10A106KP8NNNC" H 3150 2550 60  0001 C CNN "MPN"
 	1    3150 2550
 	1    0    0    -1
@@
 F 0 "C6" H 5125 1800 50  0000 L CNN
 F 1 "0.1u" H 5125 1600 50  0000 L CNN
-F 2 "Capacitors_SMD:C_0603" H 5138 1550 50  0001 C CNN
+F 2 "Capacitors_SMD:C_0402" H 5138 1550 50  0001 C CNN
 F 3 "" H 5100 1700 50  0001 C CNN
-F 4 "2013010A" H 5100 1700 60  0001 C CNN "ElecrowPN"
+F 4 "CL05B104KO5NNNC" H 5100 1700 60  0001 C CNN "MPN"
 	1    5100 1700
 	1    0    0    -1

Commit message: Rev2
Parts:
- added D4: RB161MM-20, Diode_SMD:D_SOD-123F, symbol Device:D
- C1: footprint Capacitors_SMD:C_0603 -> Capacitor_SMD:C_0603_1608Metric; symbol C -> Device:C
- C2: footprint Capacitors_SMD:C_0603 -> Capacitor_SMD:C_0402_1005Metric; symbol C -> Device:C
- C3, C4, C5, C6: footprint Capacitors_SMD:C_0402 -> Capacitor_SMD:C_0402_1005Metric; symbol C -> Device:C
- D1, D2, D3: footprint LEDs:LED_0603 -> LED_SMD:LED_0603_1608Metric; symbol LED -> Device:LED
- F1: footprint Fuse_Holders_and_Fuses:Fuse_SMD1206_Reflow -> Fuse:Fuse_1206_3216Metric; symbol Polyfuse -> Device:Polyfuse
- J1: footprint Connectors_USB:USB_C_Receptacle_Amphenol_12401610E4-2A -> Connector_USB:USB_C_Receptacle_Amphenol_12401610E4-2A; symbol USB_C_Receptacle -> Connector:USB_C_Receptacle
- J2: footprint Pin_Headers:Pin_Header_Straight_1x12 -> guri-lib:ProMicro_LeftPinhead; symbol Conn_01x12 -> Connector_Generic:Conn_01x12
- J3: footprint Pin_Headers:Pin_Header_Straight_1x12 -> guri-lib:ProMicro_RightPinhead; symbol Conn_01x12 -> Connector_Generic:Conn_01x12
- R1, R2, R7, R8: footprint Resistors_SMD:R_0603 -> Resistor_SMD:R_0402_1005Metric; symbol R -> Device:R
- R3, R4, R5, R6: footprint Resistors_SMD:R_0402 -> Resistor_SMD:R_0402_1005Metric; symbol R -> Device:R
- U1: symbol ATmega32U4 -> guri-lib:ATmega32U4
- Y1: footprint Crystals:Crystal_SMD_SeikoEpson_FA238-4pin_3.2x2.5mm -> Crystal:Crystal_SMD_SeikoEpson_FA238-4Pin_3.2x2.5mm; symbol Crystal_GND24 -> Device:Crystal_GND24
Connections:
- net VBUS: now also U1.7 (VBUS)
- net VCC: now also D4.1 (K); no longer F1.1, U1.7 (VBUS)
- new net: D4.2 (A), F1.1
Other:
- moved on the sheet: C1

Commit message: Rev3
Parts:
- J1: footprint Connector_USB:USB_C_Receptacle_Amphenol_12401610E4-2A -> guri-lib:CX90M-16P; symbol Connector:USB_C_Receptacle -> Connector:USB_C_Receptacle_USB2.0; DigikeyPN 12401610E4#2ACT-ND -> H126318CT-ND; MF Amphenol Commercial Products -> Hirose; MPN 12401610E4#2A -> CX90M-16P
Connections:
- no-connect marks 15 -> 7
Changed lines of the file:
@@
 EESchema Schematic File Version 4
 LIBS:c-pro-micro-cache
-EELAYER 26 0
+EELAYER 29 0
 EELAYER END
 $Descr A4 11693 8268
@@
 $EndComp
 $Comp
-L Connector:USB_C_Receptacle J1
-U 1 1 5AE082B7
-P 1550 3500
-F 0 "J1" H 1150 4950 50  0000 L CNN
-F 1 "USB_C_Receptacle" H 1950 4950 50  0000 R CNN
-F 2 "Connector_USB:USB_C_Receptacle_Amphenol_12401610E4-2A" H 1700 3500 50  0001 C CNN
-F 3 "" H 1700 3500 50  0001 C CNN
-F 4 "Amphenol Commercial Products" H 1550 3500 60  0001 C CNN "MF"
-F 5 "12401610E4#2A" H 1550 3500 60  0001 C CNN "MPN"
-F 6 "12401610E4#2ACT-ND" H 1550 3500 60  0001 C CNN "DigikeyPN"
-	1    1550 3500
-	1    0    0    -1
-$EndComp
-$Comp
 L Device:R R2
 U 1 1 5AE0836E
@@
 	1    0    0    -1
 $EndComp
-NoConn ~ 2150 3500
-NoConn ~ 2150 3600
-NoConn ~ 2150 3800
-NoConn ~ 2150 3900
-NoConn ~ 2150 4100
-NoConn ~ 2150 4200
-NoConn ~ 2150 4400
-NoConn ~ 2150 4500
-NoConn ~ 2150 4800
-NoConn ~ 2150 4700
 $Comp
 L power:GND #PWR02
 U 1 1 5AE084B8
-P 1650 5300
-F 0 "#PWR02" H 1650 5050 50  0001 C CNN
-F 1 "GND" H 1650 5150 50  0000 C CNN
-F 2 "" H 1650 5300 50  0001 C CNN
-F 3 "" H 1650 5300 50  0001 C CNN
-	1    1650 5300
+P 1550 4200
+F 0 "#PWR02" H 1550 3950 50  0001 C CNN
+F 1 "GND" H 1550 4050 50  0000 C CNN
+F 2 "" H 1550 4200 50  0001 C CNN
+F 3 "" H 1550 4200 50  0001 C CNN
+	1    1550 4200
 	1    0    0    -1
 $EndComp
@@
 Connection ~ 2750 2800
 Wire Wire Line
-	1650 5100 1650 5200
-Wire Wire Line
-	1250 5200 1350 5200
-Wire Wire Line
-	1250 5200 1250 5100
-Connection ~ 1650 5200
-Wire Wire Line
-	1350 5100 1350 5200
-Connection ~ 1350 5200
-Wire Wire Line
-	1450 5200 1450 5100
-Connection ~ 1450 5200
-Wire Wire Line
-	1550 5100 1550 5200
-Connection ~ 1550 5200
+	1550 4000 1550 4100
+Connection ~ 1550 4100
+Wire Wire Line
+	1250 4000 1250 4100
 Wire Wire Line
 	2150 3100 2250 3100
@@
 Wire Wire Line
 	2250 2500 2150 2500
-Wire Wire Line
-	2250 2100 2250 2200
-Wire Wire Line
-	2150 2200 2250 2200
-Connection ~ 2250 2200
-Wire Wire Line
-	2150 2300 2250 2300
 Connection ~ 2250 2300
-Wire Wire Line
-	2150 2400 2250 2400
-Connection ~ 2250 2400
 Wire Wire Line
 	5650 2150 5000 2150
@@
 L power:PWR_FLAG #FLG026
 U 1 1 5AE0E1A5
-P 1650 5200
-F 0 "#FLG026" H 1650 5275 50  0001 C CNN
-F 1 "PWR_FLAG" H 1650 5350 50  0000 C CNN
-F 2 "" H 1650 5200 50  0001 C CNN
-F 3 "" H 1650 5200 50  0001 C CNN
-	1    1650 5200
+P 1550 4100
+F 0 "#FLG026" H 1550 4175 50  0001 C CNN
+F 1 "PWR_FLAG" H 1550 4250 50  0000 C CNN
+F 2 "" H 1550 4100 50  0001 C CNN
+F 3 "" H 1550 4100 50  0001 C CNN
+	1    1550 4100
 	0    1    1    0
 $EndComp
@@
 	2750 2800 2750 3500
 Wire Wire Line
-	1650 5200 1650 5300
-Wire Wire Line
-	1350 5200 1450 5200
-Wire Wire Line
-	1450 5200 1550 5200
-Wire Wire Line
-	1550 5200 1650 5200
+	1550 4100 1550 4200
 Wire Wire Line
 	2250 3100 2350 3100
 Wire Wire Line
 	2250 3200 2350 3200
-Wire Wire Line
-	2250 2200 2250 2300
-Wire Wire Line
-	2250 2300 2250 2400
-Wire Wire Line
-	2250 2400 2250 2500
 Wire Wire Line
 	5550 1750 5550 1850
@@
 Wire Wire Line
 	5400 2450 5650 2450
+$Comp
+L Connector:USB_C_Receptacle_USB2.0 J1
+U 1 1 5AE082B7
+P 1550 3100
+F 0 "J1" H 1200 3950 50  0000 L CNN
+F 1 "USB_C_Receptacle" H 1900 3850 50  0000 R CNN
+F 2 "guri-lib:CX90M-16P" H 1700 3100 50  0001 C CNN
+F 3 "https://www.hirose.com/product/document?clcode=CL0480-0513-0-00&productname=CX90M-16P&series=CX&documenttype=2DDrawing&lang=ja&documentid=D174082_ja" H 1700 3100 50  0001 C CNN
+F 4 "Hirose" H 1550 3100 60  0001 C CNN "MF"
+F 5 "CX90M-16P" H 1550 3100 60  0001 C CNN "MPN"
+F 6 "H126318CT-ND" H 1550 3100 60  0001 C CNN "DigikeyPN"
+	1    1550 3100
+	1    0    0    -1
+$EndComp
+Wire Wire Line
+	2250 2100 2250 2300
+Wire Wire Line
+	2250 2300 2250 2500
+Wire Wire Line
+	1250 4100 1550 4100
+NoConn ~ 2150 3600
+NoConn ~ 2150 3700
 $EndSCHEMATC
